Commit message: updated urdf model forgot elevator

File: trunk/catkin_ws/src/snap_description/urdf/elevator/elevator_link.urdf (robot description, URDF)
Before this commit: robot Elevator, 3 links, 3 joints
Links:
- link elevator_arm_adapter_link: geometry collision box size=0.025 0.075 0.1; visual box size=0.025 0.075 0.1
Joints:
- joint Slider: type prismatic -> fixed
- joint arm_adapter: origin xyz=0 0.025 0 rpy=0 0 0 -> xyz=0.025 0 0 rpy=0 0 0
- joint elevator_base: origin xyz=0.0508 0 0.3937 rpy=0 0 -1.571 -> xyz=0.0508 0 0.3937 rpy=0 0 0
