Commit message: elevator urdf updated

File: trunk/catkin_ws/src/snap_description/urdf/elevator/elevator_link.xacro (robot description, xacro)
@@ -2,5 +2,5 @@
 <robot xmlns:xacro="http://ros.org/wiki/xacro">
   <xacro:property name="M_PI" value="3.1412" />
-  <xacro:property name="height" value="0.78" />
+  <xacro:property name="height_El" value="0.84455" />
   <xacro:macro name="elevator" params="parent *origin">
 <!--' every urdf should have a base link '-->
@@ -9,10 +9,10 @@
      <origin xyz="0 0 0.5" rpy="0 0 0"/>
      <mass value="1"/>
-     <inertia ixx="100"  ixy="0"  ixz="0" iyy="100" iyz="0" izz="100" />
+     <inertia ixx="10"  ixy="0"  ixz="0" iyy="10" iyz="0" izz="10" />
    </inertial>
    <visual>
      <origin xyz="0 0 0" rpy="0 0 0" />
      <geometry>
-       <box size="0.025 0.025 0.7874" />
+       <box size="0.025 0.025 ${height_El}" />
      </geometry>
      <material name="Grey">
@@ -23,5 +23,5 @@
      <origin xyz="0 0 0" rpy="0 0 0" />
      <geometry>
-       <box size="0.025 0.025 0.7874" />
+       <box size="0.025 0.025 ${height_El}" />
      </geometry>
    </collision>

Commit message: fixed urdf and elevator controller so the model displays and is controller correctly

File: trunk/catkin_ws/src/snap_description/urdf/elevator/elevator_link.xacro (robot description, xacro)
@@ -68,8 +68,8 @@
     <child link="elevator_stem_link"/>
   </joint>
-  <joint name="Slider" type="fixed">
+  <joint name="elevator_slider_link" type="prismatic"><!-- <joint name="Slider" type="fixed"> -->
     <parent link="elevator_stem_link"/>
     <child link="elevator_slider_link"/>
-    <origin xyz="0 0 0" rpy="0 0 0" />
+    <origin xyz="0 0 -${height_El/4}" rpy="0 0 0" />
     <axis xyz="0 0 1" />
     <limit lower="-0.25" upper="0.25" effort="30" velocity="0.25"/>
