Commit message: turtlebot arm is attached to the robot. files will allow other urdf changes to be made

File: trunk/catkin_ws/src/snap_description/robots/kobuki_hexagons_kinect.urdf.xacro (robot description, xacro)
@@ -10,3 +10,8 @@
   <stack_hexagons parent="base_link"/>
   <sensor_kinect  parent="base_link"/>
+  <include filename="$(find turtlebot_arm_description)/urdf/arm.xacro" />
+  <turtlebot_arm parent="base_link" color="white" gripper_color="green"
+      joints_vlimit="1.571" pan_llimit="-2.617" pan_ulimit="2.617">
+      <origin xyz="0 0 1"/>
+  </turtlebot_arm>
 </robot>

Commit message: Andrew adding snap_description to adjust kinect pose and to add the elevator. there was a conflict with the kobuku_hex... file so i just kept my version

File: trunk/catkin_ws/src/snap_description/robots/kobuki_hexagons_kinect.urdf.xacro (robot description, xacro)
@@ -7,11 +7,14 @@
 <robot name="turtlebot" xmlns:xacro="http://ros.org/wiki/xacro">
   <xacro:include filename="$(find turtlebot_description)/urdf/turtlebot_library.urdf.xacro" />
+  <!--Since we do not want to edit the turtlebot description we add the arm and elevator information here -->
+  <xacro:include filename="$(find turtlebot_arm_description)/urdf/arm.xacro" />
+  <xacro:include filename="$(find snap_description)/urdf/elevator/elevator_link" />
   <kobuki/>
   <stack_hexagons parent="base_link"/>
   <sensor_kinect  parent="base_link"/>
-  <include filename="$(find turtlebot_arm_description)/urdf/arm.xacro" />
-  <turtlebot_arm parent="base_link" color="white" gripper_color="green"
-      joints_vlimit="1.571" pan_llimit="-2.617" pan_ulimit="2.617">
-      <origin xyz="0 0 1"/>
+  <!--Attach the turtlebot arm to the elevator which connects(at this moment) to the top hexagon plate -->
+  <turtlebot_arm parent="elevator_arm_adapter_link" color="white" gripper_color="green"
+                   joints_vlimit="1.571" pan_llimit="-2.617" pan_ulimit="2.617">
+      <origin xyz="0 0.0254 0" rpy="0 1.571 1.571 "/>
   </turtlebot_arm>
 </robot>

Commit message: updated urdf model

File: trunk/catkin_ws/src/snap_description/robots/kobuki_hexagons_kinect.urdf.xacro (robot description, xacro)
@@ -16,5 +16,5 @@
   <turtlebot_arm parent="elevator_arm_adapter_link" color="white" gripper_color="green"
                    joints_vlimit="1.571" pan_llimit="-2.617" pan_ulimit="2.617">
-      <origin xyz="0 0.0254 0" rpy="0 1.571 1.571 "/>
+      <origin xyz="0.0245 0 0" rpy="1.571 0 -1.571"/>
   </turtlebot_arm>
 </robot>

Commit message: Arm should now attach in correct orientation. I tested this on my PC, but still need to verify in person. I will wait untill I am by the robot to run bringup.

File: trunk/catkin_ws/src/snap_description/robots/kobuki_hexagons_kinect.urdf.xacro (robot description, xacro)
@@ -16,5 +16,5 @@
   <turtlebot_arm parent="elevator_arm_adapter_link" color="white" gripper_color="green"
                    joints_vlimit="1.571" pan_llimit="-2.617" pan_ulimit="2.617">
-      <origin xyz="0.0245 0 0" rpy="1.571 0 -1.571"/>
+      <origin xyz="0.0245 0 0" rpy="3.142 -1.571 0"/>
   </turtlebot_arm>
 </robot>

Commit message: added two webcams to urdf and started to convert elevatorurdf to xacro. they all need to have parameters tuned

File: trunk/catkin_ws/src/snap_description/robots/kobuki_hexagons_kinect.urdf.xacro (robot description, xacro)
@@ -9,8 +9,12 @@
   <!--Since we do not want to edit the turtlebot description we add the arm and elevator information here -->
   <xacro:include filename="$(find turtlebot_arm_description)/urdf/arm.xacro" />
-  <xacro:include filename="$(find snap_description)/urdf/elevator/elevator_link.urdf" />
+  <xacro:include filename="$(find snap_description)/urdf/elevator/elevator_link.xacro" />
+  <xacro:include filename="$(find turtlebot_description)/urdf/sensors/webcamera.xacro" />
   <kobuki/>
   <stack_hexagons parent="base_link"/>
   <sensor_kinect  parent="base_link"/>
+  <elevator parent="plate_top_link">
+      <origin xyz="0.0508 0 0.3937" rpy="0 0 0"/>
+  </elevator>
   <!--Attach the turtlebot arm to the elevator which connects(at this moment) to the top hexagon plate -->
   <turtlebot_arm parent="elevator_arm_adapter_link" color="white" gripper_color="green"
@@ -18,3 +22,10 @@
       <origin xyz="0.0245 0 0" rpy="3.142 -1.571 0"/>
   </turtlebot_arm>
+  <!--Webcameras. Parameters need to be tuned -->
+  <webcamera parent="gripper_static_link" name="arm_cam">
+    <origin xyz="0.0254 -0.07 -0.0254"/>
+  </webcamera>
+  <webcamera parent="elevator_stem_link" name="head_cam">
+    <origin xyz="0 0 .5"/>
+  </webcamera>
 </robot>

File: trunk/catkin_ws/src/snap_description/urdf/elevator/elevator_link.xacro (robot description, xacro)
@@ -1,137 +1,83 @@
-<?xml version="1.0"?>
+<?xml version="1.0" ?>
 <robot xmlns:xacro="http://ros.org/wiki/xacro">
-  <!-- Import the constriansts and such from our xacro file -->
-  <xacro:include filename="$(find snap_description)/urdf/elevator/elevator_hardware.xacro"/>
-  <material name="white">
-    <color rgba="0.87 0.90 0.87 1.0"/>
-  </material>
-  <material name="black">
-    <color rgba="0.0 0.0 0.0 1.0"/>
-  </material>
-  <material name="green">
-    <color rgba="0.22 0.32 0.14 1.0"/>
-  </material>
-  <xacro:macro name="turtlebot_arm" params="parent color gripper_color *origin
-                                            joints_vlimit pan_llimit pan_ulimit">
-    <link name="arm_base_link" />
-    <joint name="arm_base_joint" type="fixed">
-      <insert_block name="origin" />
-      <parent link="${parent}"/>
-      <child link="arm_base_link" />
-    </joint>
-    <!-- fake gripper_link joint gives us a free servo!
-         this makes us 5DOF and saves you $44.90
-         that's a lot of coin! -->
-    <link name="gripper_link" />
-    <joint name="gripper_link_joint" type="revolute">
-      <origin xyz="0 0 .112" rpy="0 -1.57 0" />
-      <parent link="arm_wrist_flex_link"/>
-      <child link="gripper_link" />
-      <limit effort="30" velocity="1" lower="-3.14" upper="3.14"/>
-      <axis xyz="1 0 0"/>
-    </joint>
-    <!-- shoulder pan joint -->
-    <dynamixel_AX12_fixed parent="arm_base_link" name="arm_shoulder_pan_servo">
-      <origin xyz="0 0 0" rpy="${M_PI/2} 0 ${M_PI/2}"/>
-    </dynamixel_AX12_fixed>
-    <bioloid_F3_revolute parent="arm_shoulder_pan_servo_link" name="arm_shoulder_pan" color="${color}"
-                         vlimit="${joints_vlimit}" llimit="${pan_llimit}" ulimit="${pan_ulimit}">
-      <origin xyz="0 ${AX12_WIDTH/2} 0" rpy="${-M_PI/2} ${M_PI/2} ${M_PI}" />
-    </bioloid_F3_revolute>
-    <!-- shoulder lift joint -->
-    <dynamixel_AX12_fixed parent="arm_shoulder_pan_link" name="arm_shoulder_lift_servo">
-      <origin xyz="0 0 ${-AX12_HEIGHT-F10_HEIGHT+0.001}" rpy="0 ${M_PI} 0" />
-    </dynamixel_AX12_fixed>
-    <bioloid_F4_revolute parent="arm_shoulder_lift_servo_link" name="arm_shoulder_lift" color="${color}"
-                         vlimit="${joints_vlimit}" llimit="-2.617" ulimit="2.617">
-      <origin xyz="0 0 0" rpy="0 0 0" />
-    </bioloid_F4_revolute>
-    <bioloid_F10_fixed parent="arm_shoulder_lift_link" name="arm_shoulder_F10_0" color="${color}">
-      <origin xyz="0 0 ${F4_HEIGHT+F10_HEIGHT/2}" rpy="0 0 0" />
-    </bioloid_F10_fixed>
-    <bioloid_F10_fixed parent="arm_shoulder_F10_0_link" name="arm_shoulder_F10_1" color="${color}">
-      <origin xyz="0 0 ${F10_HEIGHT}" rpy="0 0 0" />
-    </bioloid_F10_fixed>
-    <bioloid_F10_fixed parent="arm_shoulder_F10_1_link" name="arm_shoulder_F10_2" color="${color}">
-      <origin xyz="0 0 ${F10_HEIGHT}" rpy="0 0 0" />
-    </bioloid_F10_fixed>
-    <bioloid_F3_fixed parent="arm_shoulder_F10_2_link" name="arm_shoulder_F3_0" color="${color}">
-      <origin xyz="0 0 ${F10_HEIGHT/2}" rpy="0 ${M_PI} 0" />
-    </bioloid_F3_fixed>
-    <!-- elbow joint -->
-    <dynamixel_AX12_fixed parent="arm_shoulder_F3_0_link" name="arm_elbow_flex_servo">
-      <origin xyz="0 0 ${-AX12_HEIGHT-F10_HEIGHT+0.001}" rpy="0 ${M_PI} 0"/>
-    </dynamixel_AX12_fixed>
-    <bioloid_F4_revolute parent="arm_elbow_flex_servo_link" name="arm_elbow_flex" color="${color}"
-                         vlimit="${joints_vlimit}" llimit="-2.617" ulimit="2.617">
-      <origin xyz="0 0 0" rpy="0 0 0" />
-    </bioloid_F4_revolute>
-    <bioloid_F10_fixed parent="arm_elbow_flex_link" name="arm_elbow_F10_0" color="${color}">
-      <origin xyz="0 0 ${F4_HEIGHT+F10_HEIGHT/2}" rpy="0 0 0" />
-    </bioloid_F10_fixed>
-    <bioloid_F10_fixed parent="arm_elbow_F10_0_link" name="arm_elbow_F10_1" color="${color}">
-      <origin xyz="0 0 ${F10_HEIGHT}" rpy="0 0 0" />
-    </bioloid_F10_fixed>
-    <bioloid_F10_fixed parent="arm_elbow_F10_1_link" name="arm_elbow_F10_2" color="${color}">
-      <origin xyz="0 0 ${F10_HEIGHT}" rpy="0 0 0" />
-    </bioloid_F10_fixed>
-    <bioloid_F3_fixed parent="arm_elbow_F10_2_link" name="arm_elbow_F3_0" color="${color}">
-      <origin xyz="0 0 ${F10_HEIGHT/2}" rpy="0 ${M_PI} 0" />
-    </bioloid_F3_fixed>
-    <!-- wrist joint -->
-    <dynamixel_AX12_fixed parent="arm_elbow_F3_0_link" name="arm_wrist_flex_servo">
-      <origin xyz="0 0 ${-AX12_HEIGHT-F10_HEIGHT+0.001}" rpy="0 ${M_PI} 0"/>
-    </dynamixel_AX12_fixed>
-    <bioloid_F2_revolute parent="arm_wrist_flex_servo_link" name="arm_wrist_flex" color="${color}"
-                         vlimit="${joints_vlimit}" llimit="-1.745" ulimit="1.745">
-      <origin xyz="0 0 0" rpy="0 0 0" />
-    </bioloid_F2_revolute>
-    <bioloid_F3_fixed parent="arm_wrist_flex_link" name="arm_wrist_F3_0" color="${color}">
-      <origin xyz="0 0.016 ${F2_HEIGHT}" rpy="0 ${M_PI} ${-M_PI/2}" />
-    </bioloid_F3_fixed>
-    <!-- gripper joint -->
-    <dynamixel_AX12_fixed parent="arm_wrist_F3_0_link" name="gripper_servo">
-      <origin xyz="-0.02275 0 ${-AX12_WIDTH/2}" rpy="${M_PI} ${M_PI/2} 0"/>
-    </dynamixel_AX12_fixed>
-    <!-- finger 1 -->
-    <joint name="gripper_joint" type="revolute">
-      <origin xyz="0 0 0" rpy="0 0 0"/>
-      <axis xyz="0 1 0"/>
-      <limit effort="30" velocity="0.785" lower="-0.40" upper="0.46" />
-      <parent link="gripper_servo_link"/>
-      <child link="gripper_active_link" />
-    </joint>
-    <link name="gripper_active_link">
-      <inertial>
-        <mass value="0.00001" />
-        <origin xyz="0 0 0" />
-        <inertia ixx="1.0" ixy="0.0" ixz="0.0"
-          iyy="1.0" iyz="0.0"
-          izz="1.0" />
-      </inertial>
-      <visual>
-        <origin xyz=" 0 0 0 " rpy="0 0 0" />
-        <geometry>
-          <mesh filename="package://turtlebot_arm_description/meshes/F2.stl" scale="${M_SCALE} ${M_SCALE} ${M_SCALE}"/>
-        </geometry>
-        <material name="${color}"/>
-      </visual>
-      <collision>
-        <origin xyz="0.0 0.0 0.00775" rpy="0 0 0" />
-        <geometry>
-          <box size="0.025 0.0485 0.0375"/>
-        </geometry>
-      </collision>
-    </link>
-    <finger_fixed parent="gripper_active_link" name="gripper_active_finger" color="${gripper_color}">
-      <origin xyz="0 0 ${F2_HEIGHT}" rpy="0 0 0" />
-    </finger_fixed>
-    <!-- finger 2 -->
-    <bioloid_F3_fixed parent="gripper_servo_link" name="gripper_static" color="${color}">
-      <origin xyz="0 0 ${-AX12_HEIGHT-F10_HEIGHT+0.001}" rpy="0 ${M_PI} 0" />
-    </bioloid_F3_fixed>
-    <finger_fixed parent="gripper_static_link" name="gripper_static_finger" color="${gripper_color}">
-      <origin xyz="0 0 0" rpy="0 0 ${M_PI}" />
-    </finger_fixed>
+  <xacro:property name="M_PI" value="3.1412" />
+  <xacro:property name="height" value="0.78" />
+  <xacro:macro name="elevator" params="parent *origin">
+<!--' every urdf should have a base link '-->
+<link name="elevator_stem_link">
+<inertial>
+     <origin xyz="0 0 0.5" rpy="0 0 0"/>
+     <mass value="1"/>
+     <inertia ixx="100"  ixy="0"  ixz="0" iyy="100" iyz="0" izz="100" />
+   </inertial>
+   <visual>
+     <origin xyz="0 0 0" rpy="0 0 0" />
+     <geometry>
+       <box size="0.025 0.025 0.7874" />
+     </geometry>
+     <material name="Grey">
+       <color rgba="0 1.0 1.0 1.0"/>
+     </material>
+   </visual>
+   <collision>
+     <origin xyz="0 0 0" rpy="0 0 0" />
+     <geometry>
+       <box size="0.025 0.025 0.7874" />
+     </geometry>
+   </collision>
+ </link>
+<link name="elevator_slider_link">
+   <visual>
+     <origin xyz="0 0 0" rpy="0 0 0" />
+     <geometry>
+       <box size="0.025 0.025 0.1" />
+     </geometry>
+     <material name="White">
+       <color rgba="0 0 0 1.0"/>
+     </material>
+   </visual>
+ </link>
+<link name="elevator_arm_adapter_link">
+<inertial>
+     <origin xyz="0 0 0.5" rpy="0 0 0"/>
+     <mass value="1"/>
+     <inertia ixx="100"  ixy="0"  ixz="0" iyy="100" iyz="0" izz="100" />
+   </inertial>
+   <visual>
+     <origin xyz="0 0 0" rpy="0 0 0" />
+     <geometry>
+       <box size="0.025 0.075 0.1" />
+     </geometry>
+     <material name="White">
+       <color rgba="0 1.0 1.0 1.0"/>
+     </material>
+   </visual>
+   <collision>
+     <origin xyz="0 0 0" rpy="0 0 0" />
+     <geometry>
+       <box size="0.025 0.075 0.1" />
+     </geometry>
+   </collision>
+ </link>
+<!-- Change below to alter where the elevator will attach to on the turtlebot. xacro should replace the base_link and constants for location -->
+   <joint name="elevator_base" type="fixed">
+    <!-- <origin xyz="0.025 0 0.825"/> -->
+    <!-- <parent link="base_link"/> -->
+    <insert_block name="origin" />
+    <parent link="${parent}"/>
+    <child link="elevator_stem_link"/>
+  </joint>
+  <joint name="Slider" type="fixed">
+    <parent link="elevator_stem_link"/>
+    <child link="elevator_slider_link"/>
+    <origin xyz="0 0 0" rpy="0 0 0" />
+    <axis xyz="0 0 1" />
+    <limit lower="-0.25" upper="0.25" effort="30" velocity="0.25"/>
+  </joint>
+  <joint name="arm_adapter" type="fixed">
+    <parent link="elevator_slider_link"/>
+    <child link="elevator_arm_adapter_link"/>
+    <origin xyz="0.025 0 0" rpy="0 0 0" />
+  </joint>
   </xacro:macro>
 </robot>

Commit message: updated xacro files to better reflect position of camera. urdf looks fine in rviz using roslaunch urdf_tutorial display.launch model:=<<urdf_file>> gui:=True

File: trunk/catkin_ws/src/snap_description/robots/kobuki_hexagons_kinect.urdf.xacro (robot description, xacro)
@@ -27,6 +27,7 @@
 </webcamera>
   <!-- rpy="1.5708 -0.345 0" rotated on its side and tilted up about 20 degrees -->
+  <!-- rpy="1.5708 -1.222 0" rotated on its side and tilted up about 70 degrees so the optical Z axis is pointing out of the lens -->
   <webcamera parent="elevator_stem_link" name="head_cam">
-    <origin xyz="0 0 .5"/>
+    <origin xyz="0 0 .5" rpy="-1.571 -1.222 0 "/>
   </webcamera>
 </robot>

File: trunk/catkin_ws/src/snap_description/robots/robot.urdf (robot description, URDF)
Before this commit: robot turtlebot, 65 links, 64 joints
Joints:
- joint head_cam_frame_joint: origin xyz=0 0 .5 -> xyz=0 0 .5 rpy=-1.571 -1.222 0 

Commit message: updated some positions of parts. arm camera still needs to be positioned and the location of the arm away from the elevator

File: trunk/catkin_ws/src/snap_description/robots/kobuki_hexagons_kinect.urdf.xacro (robot description, xacro)
@@ -15,13 +15,13 @@
   <sensor_kinect  parent="base_link"/>
   <elevator parent="plate_top_link">
-      <origin xyz="0.0508 0 0.3937" rpy="0 0 0"/>
+      <origin xyz="0.0508 0 ${height_El/2}" rpy="0 0 0"/>
   </elevator>
   <!--Attach the turtlebot arm to the elevator which connects(at this moment) to the top hexagon plate -->
   <turtlebot_arm parent="elevator_arm_adapter_link" color="white" gripper_color="green"
                    joints_vlimit="1.571" pan_llimit="-2.617" pan_ulimit="2.617">
-      <origin xyz="0.0245 0 0" rpy="3.142 -1.571 0"/>
+      <origin xyz="0.0889 0 0" rpy="3.142 -1.571 0"/>
   </turtlebot_arm>
   <!--Webcameras. Parameters need to be tuned -->
-  <webcamera parent="gripper_static_link" name="arm_cam">
+  <webcamera parent="arm_wrist_F3_0_link" name="arm_cam">
     <origin xyz="0.0254 -0.07 -0.0254"/>
 </webcamera>
@@ -29,5 +29,5 @@
   <!-- rpy="1.5708 -1.222 0" rotated on its side and tilted up about 70 degrees so the optical Z axis is pointing out of the lens -->
   <webcamera parent="elevator_stem_link" name="head_cam">
-    <origin xyz="0 0 .5" rpy="-1.571 -1.222 0 "/>
+    <origin xyz="-0.06985 0 ${height_El/2 + 0.2413}" rpy="-1.571 -1.222 0 "/>
   </webcamera>
 </robot>

File: trunk/catkin_ws/src/snap_description/robots/robot.urdf (robot description, URDF)
Before this commit: robot turtlebot, 65 links, 64 joints
Links:
- link elevator_stem_link: geometry collision box size=0.025 0.025 0.84455; visual box size=0.025 0.025 0.84455
Joints:
- joint arm_base_joint: origin xyz=0.0245 0 0 rpy=3.142 -1.571 0 -> xyz=0.0889 0 0 rpy=3.142 -1.571 0
- joint arm_cam_frame_joint: parent gripper_static_link -> arm_wrist_F3_0_link
- joint elevator_base: origin xyz=0.0508 0 0.3937 rpy=0 0 0 -> xyz=0.0508 0 0.422275 rpy=0 0 0
- joint head_cam_frame_joint: origin xyz=0 0 .5 rpy=-1.571 -1.222 0  -> xyz=-0.06985 0 0.663575 rpy=-1.571 -1.222 0 
